File: pcb/main.kicad_sch (KiCad schematic)
At the start: 26 parts, among them J1 out+, J2 out-, J3 RP2040, J4 Conn_01x12_Socket, J5 Conn_01x12_Socket, SW1 SW_Push, U1 DRV2605LDGS

Commit message: schematic draft
Parts:
- removed J3: RP2040, zzkeeb:MCU_rp2040-helios, symbol zzkeeb:MCU_rp2040-promicro-extend
- removed SW1: SW_Push, zzkeeb:Button_SW_SPST_SKQG_WithoutStem, symbol Switch:SW_Push
- added BOOT1: SW_Push, zzkeeb:Button_SW_SPST_SKQG_WithoutStem, symbol Switch:SW_Push
- added C1, C5, C6, C7, C8, C9: 100nF, Capacitor_SMD:C_0402_1005Metric, symbol Device:C
- added C10: 100nF, Capacitor_SMD:C_0402_1005Metric, symbol Device:C_Small
- added C11, C12: 1uF, Capacitor_SMD:C_0402_1005Metric, symbol Device:C
- added C4: 10uF, Capacitor_SMD:C_0603_1608Metric, symbol Device:C
- added F1: 500mA, Fuse:Fuse_1206_3216Metric, symbol Device:Polyfuse
- added J6: USB_C_Receptacle_USB2.0, zzkeeb:Connector_USB-C-mid-mount-ali, symbol Connector:USB_C_Receptacle_USB2.0
- added R3, R4: 5.1k, Resistor_SMD:R_0402_1005Metric, symbol Device:R
- added R5: 10k, Resistor_SMD:R_0402_1005Metric, symbol Device:R
- added U2: STM32F072CBT6, Package_QFP:LQFP-48_7x7mm_P0.5mm, symbol MCU_ST_STM32F0:STM32F072CBTx
- added U3: PRTR5V0U2X, Package_TO_SOT_SMD:SOT-143, symbol Power_Protection:PRTR5V0U2X
- added U4: XC6206P332, Package_TO_SOT_SMD:SOT-23, symbol kicad-keyboard-parts:XC6206PxxxMR-Regulator_Linear
Connections:
- net +5V: now also C1.1, C11.1, F1.2, U3.4 (VCC), U4.3 (VI)
- net GND: now also C1.2, C10.2, C11.2, C12.2, C4.2, C5.2, C6.2, C7.2, C8.2, C9.2, J6.A1 (GND), J6.A12 (GND), J6.B1 (GND), J6.B12 (GND), J6.S1 (SHIELD), R3.1, R4.2, R5.2, U2.23 (VSS), U2.35 (VSS), U2.47 (VSS), U2.8 (VSSA), U3.1 (GND), U4.1 (GND)
- net LED_OUT: now also U2.20 (PB2)
- net SCL: now also U2.42 (PB6)
- net SDA: now also U2.43 (PB7)
- net SPI_CLK: now also U2.39 (PB3)
- net SPI_MISO: now also U2.40 (PB4)
- net SPI_MOSI: now also U2.41 (PB5)
- net VIK1_CS: now also U2.45 (PB8)
- net VIK1_GPIO1: now also U2.29 (PA8)
- net VIK1_GPIO2: now also U2.30 (PA9)
- net VIK2_CS: now also U2.46 (PB9)
- net VIK2_GPIO1: now also U2.31 (PA10); no longer RE1.B
- net VIK2_GPIO2: now also U2.38 (PA15); no longer RE1.A
- net col0: now also J4.1 (Pin_1), J5.1 (Pin_1), U2.21 (PB10); no longer J4.6 (Pin_6), J5.6 (Pin_6)
- net col1: now also J4.2 (Pin_2), J5.2 (Pin_2), U2.22 (PB11); no longer J4.5 (Pin_5), J5.5 (Pin_5)
- net col2: now also J4.3 (Pin_3), J5.3 (Pin_3), U2.25 (PB12); no longer J4.4 (Pin_4), J5.4 (Pin_4)
- net col3: now also J4.4 (Pin_4), J5.4 (Pin_4), U2.26 (PB13); no longer J4.3 (Pin_3), J5.3 (Pin_3)
- net col4: now also J4.5 (Pin_5), J5.5 (Pin_5), U2.27 (PB14); no longer J4.2 (Pin_2), J5.2 (Pin_2)
- net row0: now also J4.7 (Pin_7), U2.10 (PA0); no longer J4.11 (Pin_11)
- net row1: now also J4.8 (Pin_8), U2.11 (PA1); no longer J4.10 (Pin_10)
- net row2: now also U2.12 (PA2)
- net row3: now also J4.10 (Pin_10), U2.13 (PA3); no longer D1.1 (K), J4.8 (Pin_8)
- net row4: now also J4.11 (Pin_11), U2.14 (PA4); no longer J5.11 (Pin_11)
- net row5: now also D1.1 (K), J4.12 (Pin_12), U2.3 (PC14); no longer J5.10 (Pin_10)
- net row6: now also J5.7 (Pin_7), U2.15 (PA5); no longer J5.9 (Pin_9)
- net row7: now also U2.16 (PA6)
- net row11: now reaches J5.12 (Pin_12)
- net row11: now also U2.4 (PC15)
- new net: J6.A5 (CC1), R3.2
- new net: J6.B5 (CC2), R4.1
- new net +3V3: BOOT1.1, C12.1, C4.1, C5.1, C6.1, C7.1, C8.1, C9.1, U2.1 (VBAT), U2.24 (VDD), U2.36 (VDDIO2), U2.48 (VDD), U2.9 (VDDA), U4.2 (VO)
- new net BOOT0: BOOT1.2, R5.1, U2.44 (BOOT0)
- new net C13: U2.2 (PC13)
- new net D+: J6.A6 (D+), J6.B6 (D+), U2.33 (PA12), U3.3 (I/O2)
- new net D-: J6.A7 (D-), J6.B7 (D-), U2.32 (PA11), U3.2 (I/O1)
- new net ENCA: RE1.A, U2.5 (PF0)
- new net ENCB: RE1.B, U2.6 (PF1)
- new net NRST: C10.1, U2.7 (NRST)
- new net SWCLK: U2.37 (PA14)
- new net SWDIO: U2.34 (PA13)
- new net VBUS: F1.1, J6.A4 (VBUS), J6.A9 (VBUS), J6.B4 (VBUS), J6.B9 (VBUS)
- new net col5: J4.6 (Pin_6), J5.6 (Pin_6), U2.28 (PB15)
- new net row10: J5.11 (Pin_11), U2.19 (PB1)
- new net row8: J5.9 (Pin_9), U2.17 (PA7)
- new net row9: J5.10 (Pin_10), U2.18 (PB0)
- no-connect marks 8 -> 3
Other:
- note added: "ADC_IN8/TIM3_CH3/TTa"
- note added: "ADC_IN9/TIM3_CH4/TTa"
- note added: "DFU Mode Select (Hold while resetting to enter DFU mode)"
- note added: "Decoupling Capacitors"
- note added: "ESD, reverse polarity, and over-current protection"
- note added: "FT"
- note added: "FT/SPI1_NSS/USART2_RX"
- note added: "FT/SWCLK/USART2_TX"
- note added: "FT/SWDIO"
- note added: "FT/TIM1_CH1"
- note added: "FT/TIM1_CH2/USART1_TX"
- note added: "FT/TIM1_CH3/USART1_RX"
- note added: "I2C1_SCL/TIM16_CH1/FTf"
- note added: "I2C1_SCL/USART1_TX/FTf"
- note added: "I2C1_SDA/TIM17_CH1/FTf"
- note added: "I2C1_SDA/USART1_RX/FTf"
- note added: "I2C2_SCL/USART3_TX/TIM2_CH3/FT"
- note added: "I2C2_SDA/USART3_RX/TIM2_CH4/FT"
- note added: "NRST has internal pull up Hold high for normal operation"
- note added: "Notes: CONSULT THE DATASHEET BEFORE USING ANY TIMER/I2C/SPI/UART/ADC PERIPHERALS FT and FTf pins are 5v tolerant, but output 3.3v levels. TIM2 is used for SYSTICK, so use other timers if possible. It is not recommended to use pins from PF or PC until thoroughly consulting the datasheet. SW Debug is on A13 and A14"
- note added: "OSC32_IN/TC"
- note added: "OSC32_OUT/TC"
- note added: "OSC_IN/FT"
- note added: "OSC_OUT/FT"
- note added: "Power Regulation"
- note added: "Pull BOOT0 high while reseting to activate DFU."
- note added: "SPI1_MISO/TIM3_CH1/FT"
- note added: "SPI1_MOSI/TIM3_CH2/FT"
- note added: "SPI1_SCK/TIM2_CH2/FT"
- note added: "SPI2_MISO/I2C2_SDA/FTf"
- note added: "SPI2_MOSI/FT"
- note added: "SPI2_NSS/FT"
- note added: "SPI2_SCK/I2C2_SCL/FTf"
- note added: "TTa/SPI1_SCK/ADC_IN5"
- note added: "TTa/TIM14_CH1/SPI1_NSS/ADC_IN4"
- note added: "TTa/TIM2_CH2/USART4_RX/ADC_IN1"
- note added: "TTa/TIM2_CH3/USART2_TX/ADC_IN2"
- note added: "TTa/TIM2_CH4/USART2_RX/ADC_IN3"
- note added: "TTa/TIM3_CH1/SPI1_MISO/ADC_IN6"
- note added: "TTa/TIM3_CH2/SPI1_MOSI/ADC_IN7"
- note added: "TTa/USART4_TX/ADC_IN0"
- note added: "USB-C 2.0 Port 5.1k resistors to GND on both CC pins indicate that this device is acting in legacy 2.0 UFP mode."
- note added: "WKUP2/TC"
- moved on the sheet: C2, C3, D1, H1, H2, H3, H4, J1, J2, J4, J5, JP1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
