File: pcb/main.kicad_pcb (KiCad board)
At the start: 2 copper layers, 74 x 42 mm, 26 parts, among them J1 out+, J2 out-, J3 RP2040, J4 Conn_01x12_Socket, J5 Conn_01x12_Socket, SW1 SW_Push, U1 DRV2605LDGS

Commit message: small updates
Parts:
- JP1, JP2, JP4, JP5: value VIK 5V -> 5V
Routing:
- net SCL: track 182.3 -> 189.4 mm
- net SDA: track 160.7 -> 167.0 mm
- net +5V: track 124.5 -> 128.4 mm
- net col0: track 67.5 -> 70.8 mm
- net col1: track 74.2 -> 77.5 mm
- net row7: track 25.9 -> 28.2 mm
- net VIK2_GPIO1: track 88.2 -> 90.4 mm
- net VIK2_CS: track 102.1 -> 104.1 mm
- net row0: track 25.1 -> 27.0 mm
- net col4: track 80.9 -> 82.6 mm
- net SPI_CLK: track 91.8 -> 93.2 mm
- net VIK1_CS: track 52.3 -> 53.7 mm
- net row6: track 24.8 -> 26.0 mm
- net row1: track 23.8 -> 25.0 mm
- net col2: track 74.6 -> 75.7 mm
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Other:
- board text added: "JLCJLCJLCJLC"
- board text added: "github.com/zzeneg/trio"

Commit message: jumpers for VIK GPIO, small side updates
Parts:
- added JP6: SolderJumper_3_Open, Jumper:SolderJumper-3_P1.3mm_Open_Pad1.0x1.5mm, B.Cu at (166.0, 80.0)
- added JP7: SolderJumper_3_Open, Jumper:SolderJumper-3_P1.3mm_Open_Pad1.0x1.5mm, B.Cu at (170.0, 80.0)
- turned D1 to 0 degrees
- renumbered SW1 to RST1
Connections:
- J3 pad 25: VIK2_GPIO1 -> VIK2_GPIO1/ENCB
- J3 pad 26: VIK2_GPIO2 -> VIK2_GPIO2/ENCA
- RE1 pad A: VIK2_GPIO2 -> ENCA
- RE1 pad B: VIK2_GPIO1 -> ENCB
Routing:
- net VIK2_GPIO2/ENCA: track 0.00 -> 45.2 mm, vias 0 -> 1
- net VIK2_GPIO1: track 90.4 -> 45.7 mm
- net VIK2_GPIO2: track 75.0 -> 32.5 mm, vias 2 -> 1
- net VIK2_GPIO1/ENCB: track 0.00 -> 41.3 mm
- net ENCB: track 0.00 -> 7.13 mm
- net ENCA: track 0.00 -> 6.41 mm
- net row3: track 57.8 -> 53.4 mm
- net Net-(D1-A): track 21.8 -> 25.9 mm
- net SPI_CLK: track 93.2 -> 89.8 mm
- net GND: track 60.3 -> 61.9 mm
- net col1: track 77.5 -> 76.5 mm
- net LED_OUT: track 138.2 -> 139.0 mm
- net +5V: track 128.4 -> 129.2 mm
- net SCL: track 189.4 -> 190.1 mm
- net SDA: track 167.0 -> 167.5 mm
Other:
- board text added: "ENCODER"
- board text added: "VIK2 GPIO"
- board text added: "choose:"
